Commit message: school

File: urdf/robo.xacro (robot description, xacro)
@@ -11,5 +11,5 @@
   </material>
   <xacro:macro name="wheel_macro" params="parent prefix xyz">
-    <joint name="${prefix}_joint" type="continuous">
+    <joint name="${prefix}_joint" type="fixed">
       <origin xyz="${xyz}" rpy="${radians(-90)} 0 0"/>
       <parent link="${parent}"/>
