Commit message: school

File: urdf/robo_gazebo.xacro (robot description, xacro)
@@ -11,5 +11,5 @@
   </material>
   <xacro:macro name="wheel_macro" params="parent prefix xyz">
-    <joint name="${prefix}_joint" type="fixed">
+    <joint name="${prefix}_joint" type="continuous">
       <origin xyz="${xyz}" rpy="${radians(-90)} 0 0"/>
       <parent link="${parent}"/>
@@ -18,4 +18,9 @@
     </joint>
     <link name="${prefix}_link">
+      <inertial>
+       <origin xyz="0 0 0" rpy="0 0 0"/>
+       <mass value="0.1"/>
+       <inertia ixx="0.0001" ixy="0.0" ixz="0.0" iyy="0.0001" iyz="0.0" izz="0.0001"/>
+      </inertial>
       <visual>
         <geometry>
@@ -24,5 +29,13 @@
         <material name="red"/>
       </visual>
+      <collision>
+       <geometry>
+        <cylindey radius="0.1" length="0.05"/>
+       </geometry>
+      </collision>
     </link>
+    <gazebo reference="${prefix}_link">
+     <material>Gazebo/Red</material>
+    </gazebo>
   </xacro:macro>
   <link name="world"/>
@@ -30,7 +43,12 @@
     <parent link="world"/>
     <child  link="body_link"/>
-    <origin xyz="-0.07 0 0.07" rpy="0 0 0"/>
+    <origin xyz="0.1 0 0.1" rpy="0 0 0"/>
   </joint>
   <link name="body_link">
+    <inertial>
+     <origin xyz="0 0 0" rpy="0 0 0"/>
+     <mass value="1.0"/>
+     <inertia ixx="0.001" ixy="0.0" ixz="0.0" iyy="0.001" iyz="0.0" izz="0.001"/>
+    </inertial>
     <visual>
       <origin xyz="0 0 0" rpy="0 0 0" />
@@ -40,5 +58,14 @@
       <material name="gray" />
     </visual>
+    <collision>
+     <origin xyz="0 0 0" rpy="0 0 0"/>
+     <geometry>
+      <box size="0.4 0.2 0.1"/>
+     </geometry>
+    </collision>
   </link>
+  <gazebo reference="body_link">
+   <material>Gazebo/Gray</material>
+  </gazebo>
   <xacro:wheel_macro prefix="left_wheel"  parent="body_link" xyz="-0.1 0.13 0"/>
   <xacro:wheel_macro prefix="right_wheel" parent="body_link" xyz="-0.1 -0.13 0"/>
@@ -56,4 +83,14 @@
      <material name="green" />
    </visual>
+   <collision>
+    <origin xyz="0 0 0" rpy="0 0 0"/>
+    <geometry>
+     <sphere radius="0.04"/>
+    </geometry>
+    <material name="gray"/>
+   </collision>
   </link>
+  <gazebo reference="ball_link">
+   <material>Gazebo/Gray</material>
+  </gazebo>
 </robot>

File: urdf/robo_rviz.xacro (robot description, xacro)
@@ -30,5 +30,5 @@
     <parent link="world"/>
     <child  link="body_link"/>
-    <origin xyz="-0.07 0 0.07" rpy="0 0 0"/>
+    <origin xyz="0 0 0.1" rpy="0 0 0"/>
   </joint>
   <link name="body_link">

Commit message: home

File: urdf/robo_gazebo.xacro (robot description, xacro)
@@ -31,5 +31,5 @@
       <collision>
        <geometry>
-        <cylindey radius="0.1" length="0.05"/>
+        <cylinder radius="0.1" length="0.05"/>
        </geometry>
       </collision>
@@ -39,9 +39,32 @@
     </gazebo>
   </xacro:macro>
+  <xacro:macro name="ball_macro" params="parent prefix xyz">
+   <joint name="${prefix}_joint" type="fixed">
+     <parent link="${parent}"/>
+     <child  link="${prefix}_link"/>
+     <origin xyz="${xyz}" rpy="0 0 0"/>
+   </joint>
+   <link name="${prefix}_link">
+    <visual>
+      <origin xyz="0 0 0" rpy="0 0 0" />
+      <geometry>
+        <sphere radius="0.04" />
+      </geometry>
+      <material name="green" />
+    </visual>
+    <collision>
+     <origin xyz="0 0 0" rpy="0 0 0"/>
+     <geometry>
+      <sphere radius="0.04"/>
+     </geometry>
+     <material name="gray"/>
+    </collision>
+   </link>
+  </xacro:macro>
   <link name="world"/>
   <joint name="body_joint" type="fixed">
     <parent link="world"/>
     <child  link="body_link"/>
-    <origin xyz="0.1 0 0.1" rpy="0 0 0"/>
+    <origin xyz="0 0 0.1" rpy="0 0 0"/>
   </joint>
   <link name="body_link">
@@ -68,27 +91,8 @@
    <material>Gazebo/Gray</material>
   </gazebo>
-  <xacro:wheel_macro prefix="left_wheel"  parent="body_link" xyz="-0.1 0.13 0"/>
-  <xacro:wheel_macro prefix="right_wheel" parent="body_link" xyz="-0.1 -0.13 0"/>
-  <joint name="ball_joint" type="fixed">
-    <parent link="body_link"/>
-    <child  link="ball_link"/>
-    <origin xyz="0.15 0 -0.05" rpy="0 0 0"/>
-  </joint>
-  <link name="ball_link">
-   <visual>
-     <origin xyz="0 0 0" rpy="0 0 0" />
-     <geometry>
-       <sphere radius="0.04" />
-     </geometry>
-     <material name="green" />
-   </visual>
-   <collision>
-    <origin xyz="0 0 0" rpy="0 0 0"/>
-    <geometry>
-     <sphere radius="0.04"/>
-    </geometry>
-    <material name="gray"/>
-   </collision>
-  </link>
+  <xacro:wheel_macro prefix="left_wheel"  parent="body_link" xyz="0 0.13 0"/>
+  <xacro:wheel_macro prefix="right_wheel" parent="body_link" xyz="0 -0.13 0"/>
+  <xacro:ball_macro prefix="front_caster" parent="body_link" xyz="0.15 0 -0.05"/>
+  <xacro:ball_macro prefix="back_caster" parent="body_link" xyz="-0.15 0 -0.05"/>
   <gazebo reference="ball_link">
    <material>Gazebo/Gray</material>

Commit message: home

File: urdf/robo_gazebo.xacro (robot description, xacro)
@@ -1,4 +1,4 @@
 <?xml version="1.0"?>
-<robot name="dtw_robot" xmlns:xacro="http://ros.org/wiki/xacro">
+<robot name="robo_gazebo" xmlns:xacro="http://ros.org/wiki/xacro">
   <material name="gray">
     <color rgba="0.5 0.5 0.5 2"/>
@@ -16,5 +16,17 @@
       <child  link="${prefix}_link"/>
       <axis xyz="0 0 1" />
+      <limit velocity="12.0" effort="0.4"/>
+      <dynamics damping="0.1"/>
     </joint>
+    <transmission name="${prefix}_trans" type="SimpleTransmission">
+      <type>transmission_interface/SimpleTransmission</type>
+      <joint name="${prefix}_joint">
+        <hardwareInterface>hardware_interface/VelocityJointInterface</hardwareInterface>
+      </joint>
+      <actuator name="${prefix}_motor">
+        <hardwareInterface>hardware_interface/VelocityJointInterface</hardwareInterface>
+        <mechanicalReduction>1</mechanicalReduction>
+      </actuator>
+    </transmission>
     <link name="${prefix}_link">
       <inertial>
@@ -37,4 +49,6 @@
     <gazebo reference="${prefix}_link">
      <material>Gazebo/Red</material>
+     <mu1 value="2.5"/>
+     <mu2 value="2.5"/>
     </gazebo>
   </xacro:macro>
@@ -61,7 +75,16 @@
     </collision>
    </link>
+   <gazebo reference="${prefix}_link">
+     <material>Gazebo/Green</material>
+     <mu1 value="0.5"/>
+     <mu2 value="0.5"/>
+   </gazebo>
   </xacro:macro>
+  <xacro:wheel_macro prefix="left_wheel"  parent="body_link" xyz="0 0.13 0"/>
+  <xacro:wheel_macro prefix="right_wheel" parent="body_link" xyz="0 -0.13 0"/>
+  <xacro:ball_macro prefix="front_caster" parent="body_link" xyz="0.14 0 -0.06"/>
+  <xacro:ball_macro prefix="back_caster" parent="body_link" xyz="-0.14 0 -0.06"/>
   <link name="world"/>
-  <joint name="body_joint" type="fixed">
+  <joint name="body_joint" type="planar">
     <parent link="world"/>
     <child  link="body_link"/>
@@ -91,10 +114,9 @@
    <material>Gazebo/Gray</material>
   </gazebo>
-  <xacro:wheel_macro prefix="left_wheel"  parent="body_link" xyz="0 0.13 0"/>
-  <xacro:wheel_macro prefix="right_wheel" parent="body_link" xyz="0 -0.13 0"/>
-  <xacro:ball_macro prefix="front_caster" parent="body_link" xyz="0.15 0 -0.05"/>
-  <xacro:ball_macro prefix="back_caster" parent="body_link" xyz="-0.15 0 -0.05"/>
-  <gazebo reference="ball_link">
-   <material>Gazebo/Gray</material>
+  <gazebo>
+    <plugin name="gazebo_ros_control" filename="libgazebo_ros_control.so">
+      <robotNamespace>/robo_gazebo</robotNamespace>
+      <legacyModeNS>true</legacyModeNS>
+    </plugin>
   </gazebo>
 </robot>
