Commit message: home

File: urdf/wheel_macro.xacro (robot description, xacro)
@@ -1,4 +1,6 @@
 <?xml version="1.0"?>
 <robot xmlns:xacro="http://ros.org/wiki/xacro">
+  <xacro:property name="radius" value="0.1"/>
+  <xacro:property name="length" value="0.05"/>
   <xacro:macro name="wheel_macro" params="parent prefix xyz">
     <joint name="${prefix}_joint" type="continuous">
@@ -16,5 +18,4 @@
       </joint>
       <actuator name="${prefix}_motor">
-        <hardwareInterface>hardware_interface/VelocityJointInterface</hardwareInterface>
         <mechanicalReduction>1</mechanicalReduction>
       </actuator>
@@ -28,5 +29,5 @@
       <visual>
         <geometry>
-          <cylinder radius="0.1" length="0.05" />
+          <cylinder radius="${radius}" length="${length}" />
         </geometry>
         <material name="red"/>
@@ -34,5 +35,5 @@
       <collision>
        <geometry>
-        <cylinder radius="0.1" length="0.05"/>
+        <cylinder radius="${radius}" length="${length}"/>
        </geometry>
       </collision>

Commit message: home

File: urdf/wheel_macro.xacro (robot description, xacro)
@@ -3,4 +3,5 @@
   <xacro:property name="radius" value="0.1"/>
   <xacro:property name="length" value="0.05"/>
+  <xacro:property name="mass" value="0.1"/>
   <xacro:macro name="wheel_macro" params="parent prefix xyz">
     <joint name="${prefix}_joint" type="continuous">
@@ -24,6 +25,8 @@
       <inertial>
        <origin xyz="0 0 0" rpy="0 0 0"/>
-       <mass value="0.1"/>
-       <inertia ixx="0.0001" ixy="0.0" ixz="0.0" iyy="0.0001" iyz="0.0" izz="0.0001"/>
+       <mass value="${mass}"/>
+       <inertia ixx="${mass*(3*(radius**2)+(length**2))/12}" ixy="0.0" ixz="0.0"
+                iyy="${mass*(3*(radius**2)+(length**2))/12}" iyz="0.0"
+                izz="${(mass*(radius**2))/2}"/>
       </inertial>
       <visual>
