Commit message: home

File: urdf/main_robot.xacro (robot description, xacro)
@@ -18,5 +18,7 @@
      <origin xyz="0 0 0" rpy="0 0 0"/>
      <mass value="1.0"/>
-     <inertia ixx="0.0001" ixy="0.0" ixz="0.0" iyy="0.0001" iyz="0.0" izz="0.0001"/>
+     <inertia ixx="${1.0*((0.18**2)+(0.1**2))/3}" ixy="0.0" ixz="0.0"
+              iyy="${1.0*((0.4**2)+(0.1**2))/3}" iyz="0.0"
+              izz="${1.0*((0.18**2)+(0.18*2))/3}"/>
     </inertial>
     <visual>

Commit message: home

File: urdf/main_robot.xacro (robot description, xacro)
@@ -8,7 +8,7 @@
   <xacro:ball_macro prefix="front_caster" parent="body_link" xyz="0.14 0 -0.06"/>
   <xacro:ball_macro prefix="back_caster" parent="body_link" xyz="-0.14 0 -0.06"/>
-  <link name="world"/>
-  <joint name="base_joint" type="planar">
-    <parent link="world"/>
+  <link name="base_link"/>
+  <joint name="base_joint" type="fixed">
+    <parent link="base_link"/>
     <child link="body_link"/>
     <origin xyz="0 0 0.1" rpy="0 0 0"/>

File: urdf/wheel_macro.xacro (robot description, xacro)
@@ -10,6 +10,4 @@
       <child  link="${prefix}_link"/>
       <axis xyz="0 0 1" />
-      <limit velocity="12.0" effort="0.4"/>
-      <dynamics damping="0.1"/>
     </joint>
     <transmission name="${prefix}_trans" type="SimpleTransmission">
@@ -44,6 +42,6 @@
     <gazebo reference="${prefix}_link">
      <material>Gazebo/Red</material>
-     <mu1 value="1.5"/>
-     <mu2 value="1.5"/>
+     <mu1 value="2.5"/>
+     <mu2 value="2.5"/>
     </gazebo>
   </xacro:macro>
