Commit message: school

File: urdf/main_robot_rviz.xacro (robot description, xacro)
@@ -8,5 +8,5 @@
   <xacro:ball_macro prefix="front_caster" parent="body_link" xyz="0.14 0 -0.06"/>
   <xacro:ball_macro prefix="back_caster" parent="body_link" xyz="-0.14 0 -0.06"/>
-  <!--<link name="base_link"/>
+  <link name="base_link"/>
   <joint name="base_joint" type="fixed">
     <parent link="base_link"/>
@@ -14,5 +14,4 @@
     <origin xyz="0 0 0.1" rpy="0 0 0"/>
   </joint>
--->
   <link name="body_link">
     <inertial>
